Commit message: restore the source code

File: src/dual_arm/model/dualarm_mod.urdf (robot description, URDF)
Before this commit: robot dualarm, 16 links, 15 joints
Joints:
- joint j0: origin xyz=0 0.159800001842985 0.5727 rpy=1.5707963267949 0 1.57079632679488 -> xyz=0 0.159800001842985 0.685 rpy=1.5707963267949 0 1.57079632679488

File: src/dual_arm/model/dualarm_mod_test.urdf (robot description, URDF)
Before this commit: robot dualarm, 16 links, 15 joints
Links:
- added link Hand_RF1J1, mass 0.00152598624013965; collision mesh filename=file://$(arg meshDirectory)/Hand_RF1J1.STL; visual mesh filename=file://$(arg meshDirectory)/Hand_RF1J1.STL
- added link Hand_RF1J2, mass 0.0341378762034902; collision mesh filename=file://$(arg meshDirectory)/Hand_RF1J2.STL; visual mesh filename=file://$(arg meshDirectory)/Hand_RF1J2.STL
- added link Hand_RF1J3, mass 0.017723; collision mesh filename=file://$(arg meshDirectory)/Hand_RF1J3.STL; visual mesh filename=file://$(arg meshDirectory)/Hand_RF1J3.STL
- added link Hand_RF1J4, mass 0.0098292; collision mesh filename=file://$(arg meshDirectory)/Hand_RF1J4.STL; visual mesh filename=file://$(arg meshDirectory)/Hand_RF1J4.STL
- added link Hand_RF2J1, mass 0.00152598652963305; collision mesh filename=file://$(arg meshDirectory)/Hand_RF2J1.STL; visual mesh filename=file://$(arg meshDirectory)/Hand_RF2J1.STL
- added link Hand_RF2J2, mass 0.0341378762027317; collision mesh filename=file://$(arg meshDirectory)/Hand_RF2J2.STL; visual mesh filename=file://$(arg meshDirectory)/Hand_RF2J2.STL
- added link Hand_RF2J3, mass 0.0177234171241366; collision mesh filename=file://$(arg meshDirectory)/Hand_RF2J3.STL; visual mesh filename=file://$(arg meshDirectory)/Hand_RF2J3.STL
- added link Hand_RF2J4, mass 0.00982919734972211; collision mesh filename=file://$(arg meshDirectory)/Hand_RF2J4.STL; visual mesh filename=file://$(arg meshDirectory)/Hand_RF2J4.STL
- added link Hand_RF3J1, mass 0.00152598635461991; collision mesh filename=file://$(arg meshDirectory)/Hand_RF3J1.STL; visual mesh filename=file://$(arg meshDirectory)/Hand_RF3J1.STL
- added link Hand_RF3J2, mass 0.0341378762034901; collision mesh filename=file://$(arg meshDirectory)/Hand_RF3J2.STL; visual mesh filename=file://$(arg meshDirectory)/Hand_RF3J2.STL
- added link Hand_RF3J3, mass 0.017723416829923; collision mesh filename=file://$(arg meshDirectory)/Hand_RF3J3.STL; visual mesh filename=file://$(arg meshDirectory)/Hand_RF3J3.STL
- added link Hand_RF3J4, mass 0.00982918937760021; collision mesh filename=file://$(arg meshDirectory)/Hand_RF3J4.STL; visual mesh filename=file://$(arg meshDirectory)/Hand_RF3J4.STL
- added link Hand_RT1, mass 0.0206488185480908; collision mesh filename=file://$(arg meshDirectory)/Hand_RT1.STL; visual mesh filename=file://$(arg meshDirectory)/Hand_RT1.STL
- added link Hand_RT2, mass 0.00152598624013964; collision mesh filename=file://$(arg meshDirectory)/Hand_RT2.STL; visual mesh filename=file://$(arg meshDirectory)/Hand_RT2.STL
- added link Hand_RT3, mass 0.0341378762034901; collision mesh filename=file://$(arg meshDirectory)/Hand_RT3.STL; visual mesh filename=file://$(arg meshDirectory)/Hand_RT3.STL
- added link Hand_RT4, mass 0.00982919949661632; collision mesh filename=file://$(arg meshDirectory)/Hand_RT4.STL; visual mesh filename=file://$(arg meshDirectory)/Hand_RT4.STL
- added link RHandbase_Link, mass 0.15198; collision mesh filename=file://$(arg meshDirectory)/RHandbase_Link.STL; visual mesh filename=file://$(arg meshDirectory)/RHandbase_Link.STL
- added link rh_p12_rn_base, mass 0.236; collision mesh filename=file://$(arg meshDirectory)/base.stl scale=0.001 0.001 0.001; visual mesh filename=file://$(arg meshDirectory)/base.stl scale=0.001 0.001 0.001
- added link rh_p12_rn_l1, mass 0.068; collision mesh filename=file://$(arg meshDirectory)/l1.stl scale=0.001 0.001 0.001; visual mesh filename=file://$(arg meshDirectory)/l1.stl scale=0.001 0.001 0.001
- added link rh_p12_rn_l2, mass 0.022; collision mesh filename=file://$(arg meshDirectory)/l2.stl scale=0.001 0.001 0.001; visual mesh filename=file://$(arg meshDirectory)/l2.stl scale=0.001 0.001 0.001
- added link rh_p12_rn_r1, mass 0.068; collision mesh filename=file://$(arg meshDirectory)/r1.stl scale=0.001 0.001 0.001; visual mesh filename=file://$(arg meshDirectory)/r1.stl scale=0.001 0.001 0.001
- added link rh_p12_rn_r2, mass 0.022; collision mesh filename=file://$(arg meshDirectory)/r2.stl scale=0.001 0.001 0.001; visual mesh filename=file://$(arg meshDirectory)/r2.stl scale=0.001 0.001 0.001
Joints:
- added joint LHand_joint: type fixed, parent LWrR_Link, child rh_p12_rn_base, origin xyz=-0.0177 -0.104748 0 rpy=1.5708 1.5708 0
- added joint RF1J1: type fixed, parent RHandbase_Link, child Hand_RF1J1, origin xyz=-0.006325 0.033168 -0.11515 rpy=3.1416 0 0
- added joint RF1J2: type fixed, parent Hand_RF1J1, child Hand_RF1J2, origin xyz=0 0.0004981 4.3578E-05 rpy=3.1416 -1.4835 -1.5708
- added joint RF1J3: type fixed, parent Hand_RF1J2, child Hand_RF1J3, origin xyz=0.0401 0 -0.000125 rpy=0 0 0
- added joint RF1J4: type fixed, parent Hand_RF1J3, child Hand_RF1J4, origin xyz=0.03005 0 -5E-05 rpy=0 0 0
- added joint RF2J1: type fixed, parent RHandbase_Link, child Hand_RF2J1, origin xyz=-0.006325 0 -0.1166 rpy=3.1416 0 0
- added joint RF2J2: type fixed, parent Hand_RF2J1, child Hand_RF2J2, origin xyz=0 0.0005 0 rpy=1.5708 -1.5708 0
- added joint RF2J3: type fixed, parent Hand_RF2J2, child Hand_RF2J3, origin xyz=0.0401 0 -0.000125 rpy=0 0 0
- added joint RF2J4: type fixed, parent Hand_RF2J3, child Hand_RF2J4, origin xyz=0.03005 0 -5E-05 rpy=0 0 0
- added joint RF3J1: type fixed, parent RHandbase_Link, child Hand_RF3J1, origin xyz=-0.006325 -0.033168 -0.11515 rpy=3.1416 0 0
- added joint RF3J2: type fixed, parent Hand_RF3J1, child Hand_RF3J2, origin xyz=0 0.0004981 -4.3578E-05 rpy=0 -1.4835 1.5708
- added joint RF3J3: type fixed, parent Hand_RF3J2, child Hand_RF3J3, origin xyz=0.0401 0 -0.000125 rpy=0 0 0
- added joint RF3J4: type fixed, parent Hand_RF3J3, child Hand_RF3J4, origin xyz=0.03005 0 -5E-05 rpy=0 0 0
- added joint RHBase: type fixed, parent RWrR_Link, child RHandbase_Link, origin xyz=-0.0177 -0.104748 0 rpy=-1.5708 -1.5708 0
- added joint RT1: type fixed, parent RHandbase_Link, child Hand_RT1, origin xyz=0.006325 0.010945 -0.044721 rpy=3.0543 0 3.1416
- added joint RT2: type fixed, parent Hand_RT1, child Hand_RT2, origin xyz=5E-05 0.0441 0 rpy=-1.5708 0 -3.1416
- added joint RT3: type fixed, parent Hand_RT2, child Hand_RT3, origin xyz=0 0 0 rpy=0 1.5708 1.5708
- added joint RT4: type fixed, parent Hand_RT3, child Hand_RT4, origin xyz=0.0401000000000001 0 -0.000675000000000314 rpy=0 0 0
- added joint rh_l1: type fixed, parent rh_p12_rn_base, child rh_p12_rn_l1, origin xyz=0.0 -0.008 0.048 rpy=0 0 0
- added joint rh_l2: type fixed, parent rh_p12_rn_l1, child rh_p12_rn_l2, origin xyz=0.0 -0.0493634 0.0285 rpy=0 0 0
- added joint rh_r1: type fixed, parent rh_p12_rn_base, child rh_p12_rn_r1, origin xyz=0.0 0.008 0.048 rpy=0 0 0
- added joint rh_r2: type fixed, parent rh_p12_rn_r1, child rh_p12_rn_r2, origin xyz=0.0 0.0493634 0.0285 rpy=0 0 0
- joint j0: limit lower=-0.3 upper=0.3 effort=100 velocity=10 -> lower=0.0 upper=0.6 effort=100 velocity=10; origin xyz=0 0.159800001842985 0.5727 rpy=1.5707963267949 0 1.57079632679488 -> xyz=0.1598000018429850 0 0.615 rpy=1.5707963267949 0 0
- joint j14: mimic joint=j7 multiplier=1 offset=0 -> (none)
